File: Isolated supply 12V.kicad_sch (KiCad schematic)
At the start: 6 parts, among them U31 TD6-48S15W

Commit message: Refactored top sheet
Parts:
- renumbered C51 to C50, C52 to C51, C53 to C52, C54 to C53, U31 to U30
Changed lines of the file:
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@@
   (symbol (lib_id "Device:C_Polarized") (at 113.03 90.17 0) (unit 1)
     (in_bom yes) (on_board yes) (fields_autoplaced)
-    (property "Reference" "C51" (id 0) (at 116.84 88.8999 0)
+    (property "Reference" "C50" (id 0) (at 116.84 88.8999 0)
       (effects (font (size 1.27 1.27)) (justify left))
     )
@@
   (symbol (lib_id "Device:C") (at 166.37 90.17 0) (unit 1)
     (in_bom yes) (on_board yes)
-    (property "Reference" "C53" (id 0) (at 161.29 87.63 0)
+    (property "Reference" "C52" (id 0) (at 161.29 87.63 0)
       (effects (font (size 1.27 1.27)) (justify left))
     )
@@
   (symbol (lib_id "Device:C") (at 176.53 90.17 0) (unit 1)
     (in_bom yes) (on_board yes)
-    (property "Reference" "C54" (id 0) (at 171.45 87.63 0)
+    (property "Reference" "C53" (id 0) (at 171.45 87.63 0)
       (effects (font (size 1.27 1.27)) (justify left))
     )
@@
   (symbol (lib_id "PersonnalSymbolLibrary:TD6-48S15W") (at 132.08 83.82 0) (unit 1)
     (in_bom yes) (on_board yes) (fields_autoplaced)
-    (property "Reference" "U31" (id 0) (at 139.7 78.74 0))
+    (property "Reference" "U30" (id 0) (at 139.7 78.74 0))
     (property "Value" "TD6-48S15W" (id 1) (at 139.7 81.28 0))
     (property "Footprint" "PersonnalFootprintLibrary:TD6-48S15W" (id 2) (at 142.24 104.14 0)
@@
   (symbol (lib_id "Device:C") (at 157.48 90.17 0) (unit 1)
     (in_bom yes) (on_board yes)
-    (property "Reference" "C52" (id 0) (at 151.511 87.7316 0)
+    (property "Reference" "C51" (id 0) (at 151.511 87.7316 0)
       (effects (font (size 1.27 1.27)) (justify left))
     )
