File: digital_out.kicad_sch (KiCad schematic)
At the start: 6 parts, among them Q12 AO3400A, U32 EL357N-G

Commit message: Refactored top sheet
Parts:
- renumbered D6 to D8, Q12 to Q17, R69 to R85, R70 to R86, R71 to R87, U32 to U34
Changed lines of the file:
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@@
   (symbol (lib_id "Device:R") (at 146.05 66.04 270) (unit 1)
     (in_bom yes) (on_board yes)
-    (property "Reference" "R70" (id 0) (at 146.05 63.3222 90))
+    (property "Reference" "R86" (id 0) (at 146.05 63.3222 90))
     (property "Value" "1k" (id 1) (at 146.05 68.1736 90))
     (property "Footprint" "Resistor_SMD:R_1206_3216Metric" (id 2) (at 146.05 64.262 90)
@@
   (symbol (lib_id "Device:R") (at 166.37 87.63 180) (unit 1)
     (in_bom yes) (on_board yes) (fields_autoplaced)
-    (property "Reference" "R71" (id 0) (at 168.91 86.3599 0)
+    (property "Reference" "R87" (id 0) (at 168.91 86.3599 0)
       (effects (font (size 1.27 1.27)) (justify right))
     )
@@
   (symbol (lib_id "Device:R") (at 146.05 58.42 270) (unit 1)
     (in_bom yes) (on_board yes)
-    (property "Reference" "R69" (id 0) (at 146.05 55.7022 90))
+    (property "Reference" "R85" (id 0) (at 146.05 55.7022 90))
     (property "Value" "1k" (id 1) (at 146.05 60.5536 90))
     (property "Footprint" "Resistor_SMD:R_1206_3216Metric" (id 2) (at 146.05 56.642 90)
@@
   (symbol (lib_id "PersonnalSymbolLibrary:B5819W_SL") (at 176.53 71.12 270) (unit 1)
     (in_bom yes) (on_board yes) (fields_autoplaced)
-    (property "Reference" "D6" (id 0) (at 179.07 69.8499 90)
+    (property "Reference" "D8" (id 0) (at 179.07 69.8499 90)
       (effects (font (size 1.27 1.27)) (justify left))
     )
@@
   (symbol (lib_id "Transistor_FET:AO3400A") (at 173.99 81.28 0) (unit 1)
     (in_bom yes) (on_board yes) (fields_autoplaced)
-    (property "Reference" "Q12" (id 0) (at 180.34 80.0099 0)
+    (property "Reference" "Q17" (id 0) (at 180.34 80.0099 0)
       (effects (font (size 1.27 1.27)) (justify left))
     )
@@
   (symbol (lib_id "PersonnalSymbolLibrary:EL357N-G") (at 158.75 68.58 0) (unit 1)
     (in_bom yes) (on_board yes) (fields_autoplaced)
-    (property "Reference" "U32" (id 0) (at 158.75 59.69 0))
+    (property "Reference" "U34" (id 0) (at 158.75 59.69 0))
     (property "Value" "EL357N-G" (id 1) (at 158.75 62.23 0))
     (property "Footprint" "ELM357N-G:SOP254P700X200-4N" (id 2) (at 160.02 73.66 0)
