File: isolated_inputs.kicad_sch (KiCad schematic)
At the start: 0 parts

Commit message: Refactored top sheet
Other:
- removed sheet digital_out2
- removed sheet digital_out3
Changed lines of the file:
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@@
-    (stroke (width 0) (type default) (color 0 0 0 0))
-  )
-  (wire (pts (xy 194.31 74.93) (xy 203.2 74.93))
     (stroke (width 0) (type default) (color 0 0 0 0))
   )
@@
     (stroke (width 0) (type default) (color 0 0 0 0))
   )
-  (wire (pts (xy 250.19 29.21) (xy 250.19 34.29))
-    (stroke (width 0) (type default) (color 0 0 0 0))
-  )
   (wire (pts (xy 129.54 111.76) (xy 133.35 111.76))
     (stroke (width 0) (type default) (color 0 0 0 0))
   )
-  (wire (pts (xy 236.22 36.83) (xy 248.92 36.83))
-    (stroke (width 0) (type default) (color 0 0 0 0))
-  )
   (wire (pts (xy 133.35 111.76) (xy 133.35 133.35))
     (stroke (width 0) (type default) (color 0 0 0 0))
@@
     (stroke (width 0) (type default) (color 0 0 0 0))
   )
-  (wire (pts (xy 236.22 80.01) (xy 250.19 80.01))
-    (stroke (width 0) (type default) (color 0 0 0 0))
-  )
-  (wire (pts (xy 236.22 34.29) (xy 250.19 34.29))
-    (stroke (width 0) (type default) (color 0 0 0 0))
-  )
   (wire (pts (xy 129.54 152.4) (xy 144.78 152.4))
     (stroke (width 0) (type default) (color 0 0 0 0))
@@
     (stroke (width 0) (type default) (color 0 0 0 0))
   )
-  (wire (pts (xy 236.22 74.93) (xy 250.19 74.93))
-    (stroke (width 0) (type default) (color 0 0 0 0))
-  )
   (wire (pts (xy 81.28 73.66) (xy 86.36 73.66))
     (stroke (width 0) (type default) (color 0 0 0 0))
   )
-  (wire (pts (xy 199.39 80.01) (xy 199.39 85.09))
-    (stroke (width 0) (type default) (color 0 0 0 0))
-  )
   (wire (pts (xy 86.36 88.9) (xy 59.69 88.9))
     (stroke (width 0) (type default) (color 0 0 0 0))
@@
     (stroke (width 0) (type default) (color 0 0 0 0))
   )
-  (wire (pts (xy 236.22 77.47) (xy 248.92 77.47))
-    (stroke (width 0) (type default) (color 0 0 0 0))
-  )
   (wire (pts (xy 86.36 106.68) (xy 59.69 106.68))
     (stroke (width 0) (type default) (color 0 0 0 0))
   )
-  (wire (pts (xy 194.31 34.29) (xy 203.2 34.29))
-    (stroke (width 0) (type default) (color 0 0 0 0))
-  )
   (wire (pts (xy 139.7 149.86) (xy 139.7 128.27))
     (stroke (width 0) (type default) (color 0 0 0 0))
@@
     (stroke (width 0) (type default) (color 0 0 0 0))
   )
-  (wire (pts (xy 250.19 69.85) (xy 250.19 74.93))
-    (stroke (width 0) (type default) (color 0 0 0 0))
-  )
-  (wire (pts (xy 250.19 80.01) (xy 250.19 83.82))
-    (stroke (width 0) (type default) (color 0 0 0 0))
-  )
   (wire (pts (xy 86.36 128.27) (xy 59.69 128.27))
     (stroke (width 0) (type default) (color 0 0 0 0))
@@
     (stroke (width 0) (type default) (color 0 0 0 0))
   )
-  (wire (pts (xy 236.22 39.37) (xy 250.19 39.37))
-    (stroke (width 0) (type default) (color 0 0 0 0))
-  )
-  (wire (pts (xy 250.19 39.37) (xy 250.19 43.18))
-    (stroke (width 0) (type default) (color 0 0 0 0))
-  )
   (wire (pts (xy 129.54 76.2) (xy 133.35 76.2))
     (stroke (width 0) (type default) (color 0 0 0 0))
@@
     (stroke (width 0) (type default) (color 0 0 0 0))
   )
-  (wire (pts (xy 199.39 39.37) (xy 199.39 43.18))
-    (stroke (width 0) (type default) (color 0 0 0 0))
-  )
-  (wire (pts (xy 203.2 39.37) (xy 199.39 39.37))
-    (stroke (width 0) (type default) (color 0 0 0 0))
-  )
   (wire (pts (xy 133.35 185.42) (xy 151.13 185.42))
     (stroke (width 0) (type default) (color 0 0 0 0))
@@
     (stroke (width 0) (type default) (color 0 0 0 0))
   )
-  (wire (pts (xy 203.2 80.01) (xy 199.39 80.01))
-    (stroke (width 0) (type default) (color 0 0 0 0))
-  )
   (hierarchical_label "LIMZ_NPN_PIN" (shape input) (at 81.28 57.15 180)
     (effects (font (size 1.27 1.27)) (justify right))
   )
-  (hierarchical_label "GND_ISO" (shape input) (at 250.19 43.18 270)
-    (effects (font (size 1.27 1.27)) (justify right))
-  )
-  (hierarchical_label "FLOOD_ISO" (shape output) (at 248.92 36.83 0)
-    (effects (font (size 1.27 1.27)) (justify left))
-  )
-  (hierarchical_label "MIST" (shape input) (at 194.31 74.93 180)
-    (effects (font (size 1.27 1.27)) (justify right))
-  )
-  (hierarchical_label "MIST_ISO" (shape output) (at 248.92 77.47 0)
-    (effects (font (size 1.27 1.27)) (justify left))
-  )
   (hierarchical_label "LIMIT_Y_MCU" (shape output) (at 144.78 39.37 0)
     (effects (font (size 1.27 1.27)) (justify left))
   )
-  (hierarchical_label "GND_MCU" (shape input) (at 199.39 43.18 270)
-    (effects (font (size 1.27 1.27)) (justify right))
-  )
-  (hierarchical_label "GND_ISO" (shape input) (at 250.19 83.82 270)
-    (effects (font (size 1.27 1.27)) (justify right))
-  )
   (hierarchical_label "LIMX_NPN_PIN" (shape input) (at 81.28 22.86 180)
     (effects (font (size 1.27 1.27)) (justify right))
   )
-  (hierarchical_label "CYCLE_START_MCU" (shape output) (at 144.78 173.99 0)
-    (effects (font (size 1.27 1.27)) (justify left))
-  )
-  (hierarchical_label "VCC_12V_ISO" (shape input) (at 250.19 69.85 90)
+  (hierarchical_label "CYCLE_ST_MCU" (shape output) (at 144.78 173.99 0)
     (effects (font (size 1.27 1.27)) (justify left))
   )
@@
     (effects (font (size 1.27 1.27)) (justify right))
   )
-  (hierarchical_label "FEED_HOLD" (shape input) (at 81.28 130.81 180)
-    (effects (font (size 1.27 1.27)) (justify right))
-  )
-  (hierarchical_label "VCC_12V_ISO" (shape input) (at 250.19 29.21 90)
-    (effects (font (size 1.27 1.27)) (justify left))
+  (hierarchical_label "FEED_HLD" (shape input) (at 81.28 130.81 180)
+    (effects (font (size 1.27 1.27)) (justify right))
   )
   (hierarchical_label "DOOR" (shape input) (at 81.28 152.4 180)
@@
     (effects (font (size 1.27 1.27)) (justify right))
   )
-  (hierarchical_label "GND_MCU" (shape input) (at 199.39 85.09 270)
-    (effects (font (size 1.27 1.27)) (justify right))
-  )
   (hierarchical_label "PROBE_MCU" (shape output) (at 144.78 109.22 0)
     (effects (font (size 1.27 1.27)) (justify left))
   )
-  (hierarchical_label "CYCLE_START" (shape input) (at 81.28 173.99 180)
-    (effects (font (size 1.27 1.27)) (justify right))
-  )
-  (hierarchical_label "FLOOD" (shape input) (at 194.31 34.29 180)
+  (hierarchical_label "CYCLE_ST" (shape input) (at 81.28 173.99 180)
     (effects (font (size 1.27 1.27)) (justify right))
   )
@@
     (effects (font (size 1.27 1.27)) (justify left))
   )
-  (hierarchical_label "FEED_HOLD_MCU" (shape output) (at 144.78 130.81 0)
+  (hierarchical_label "FEED_HLD_MCU" (shape output) (at 144.78 130.81 0)
     (effects (font (size 1.27 1.27)) (justify left))
   )
@@
     )
   )
-  (sheet (at 203.2 72.39) (size 33.02 10.16) (fields_autoplaced)
-    (stroke (width 0.1524) (type solid) (color 0 0 0 0))
-    (fill (color 0 0 0 0.0000))
-    (property "Sheet name" "digital_out3" (id 0) (at 203.2 71.6784 0)
-      (effects (font (size 1.27 1.27)) (justify left bottom))
-    )
-    (property "Sheet file" "digital_out.kicad_sch" (id 1) (at 203.2 83.1346 0)
-      (effects (font (size 1.27 1.27)) (justify left top))
-    )
-    (pin "GND_ISO" input (at 236.22 80.01 0)
-      (effects (font (size 1.27 1.27)) (justify right))
-    )
-    (pin "INPUT" input (at 203.2 74.93 180)
-      (effects (font (size 1.27 1.27)) (justify left))
-    )
-    (pin "GND_INPUT" input (at 203.2 80.01 180)
-      (effects (font (size 1.27 1.27)) (justify left))
-    )
-    (pin "VCC_12V_ISO" input (at 236.22 74.93 0)
-      (effects (font (size 1.27 1.27)) (justify right))
-    )
-    (pin "OUTPUT" output (at 236.22 77.47 0)
-      (effects (font (size 1.27 1.27)) (justify right))
-    )
-  )
   (sheet (at 86.36 168.91) (size 43.18 10.16) (fields_autoplaced)
     (stroke (width 0.1524) (type solid) (color 0 0 0 0))
@@
       (effects (font (size 1.27 1.27)) (justify right))
     )
-  )
-  (sheet (at 203.2 31.75) (size 33.02 10.16) (fields_autoplaced)
-    (stroke (width 0.1524) (type solid) (color 0 0 0 0))
-    (fill (color 0 0 0 0.0000))
-    (property "Sheet name" "digital_out2" (id 0) (at 203.2 31.0384 0)
-      (effects (font (size 1.27 1.27)) (justify left bottom))
-    )
-    (property "Sheet file" "digital_out.kicad_sch" (id 1) (at 203.2 42.4946 0)
-      (effects (font (size 1.27 1.27)) (justify left top))
-    )
-    (pin "GND_ISO" input (at 236.22 39.37 0)
-      (effects (font (size 1.27 1.27)) (justify right))
-    )
-    (pin "INPUT" input (at 203.2 34.29 180)
-      (effects (font (size 1.27 1.27)) (justify left))
-    )
-    (pin "GND_INPUT" input (at 203.2 39.37 180)
-      (effects (font (size 1.27 1.27)) (justify left))
-    )
-    (pin "VCC_12V_ISO" input (at 236.22 34.29 0)
-      (effects (font (size 1.27 1.27)) (justify right))
-    )
-    (pin "OUTPUT" output (at 236.22 36.83 0)
-      (effects (font (size 1.27 1.27)) (justify right))
-    )
