File: isolated_rs485.kicad_sch (KiCad schematic)
At the start: 16 parts, among them U11 ADuM121N, U12 B0505S-1WR3, U13 NE555D, U14 SN75176AD

Commit message: Refactored top sheet
Parts:
- renumbered R13 to R7, R14 to R8, R15 to R9
Changed lines of the file:
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@@
   (symbol (lib_id "Device:R") (at 179.07 54.61 0) (unit 1)
     (in_bom yes) (on_board yes) (fields_autoplaced)
-    (property "Reference" "R14" (id 0) (at 181.61 53.3399 0)
+    (property "Reference" "R8" (id 0) (at 181.61 53.3399 0)
       (effects (font (size 1.27 1.27)) (justify left))
     )
@@
   (symbol (lib_id "Device:R") (at 156.21 45.72 180) (unit 1)
     (in_bom yes) (on_board yes) (fields_autoplaced)
-    (property "Reference" "R13" (id 0) (at 158.75 44.4499 0)
+    (property "Reference" "R7" (id 0) (at 158.75 44.4499 0)
       (effects (font (size 1.27 1.27)) (justify right))
     )
@@
   (symbol (lib_id "Device:R") (at 204.47 95.25 180) (unit 1)
     (in_bom yes) (on_board yes) (fields_autoplaced)
-    (property "Reference" "R15" (id 0) (at 207.01 93.9799 0)
-      (effects (font (size 1.27 1.27)) (justify right))
-    )
+    (property "Reference" "R9" (id 0) (at 207.01 93.9799 0)
+      (effects (font (size 1.27 1.27)) (justify right))
+    )
