File: microcontroller.kicad_sch (KiCad schematic)
At the start: 23 parts, among them J30 Conn_01x02, U20 W25Q128JVS, U21 RP2040, Y1 X322512MSB4SI

Commit message: Refactored top sheet
Parts:
- renumbered C25 to C24, C26 to C25, C27 to C26, C28 to C27, C29 to C28, C30 to C29, C31 to C30, C32 to C31, C33 to C32, C34 to C33, C35 to C34, C36 to C35, C37 to C36, C38 to C37, R38 to R26, R39 to R27, R40 to R28, R41 to R29, R42 to R30, U20 to U19, U21 to U20
Changed lines of the file:
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@@
   (symbol (lib_id "MCU_RaspberryPi_RP2040:RP2040") (at 172.72 105.41 0) (unit 1)
     (in_bom yes) (on_board yes)
-    (property "Reference" "U21" (id 0) (at 144.78 55.88 0))
+    (property "Reference" "U20" (id 0) (at 144.78 55.88 0))
     (property "Value" "RP2040" (id 1) (at 196.85 156.21 0))
     (property "Footprint" "MCU_RaspberryPi_and_Boards:RP2040-QFN-56" (id 2) (at 153.67 105.41 0)
@@
   (symbol (lib_id "Device:C") (at 198.12 45.72 0) (unit 1)
     (in_bom yes) (on_board yes)
-    (property "Reference" "C32" (id 0) (at 198.501 43.2816 0)
+    (property "Reference" "C31" (id 0) (at 198.501 43.2816 0)
       (effects (font (size 1.27 1.27)) (justify left))
     )
@@
   (symbol (lib_id "Device:C") (at 266.7 33.02 0) (unit 1)
     (in_bom yes) (on_board yes)
-    (property "Reference" "C38" (id 0) (at 267.97 31.1149 0)
+    (property "Reference" "C37" (id 0) (at 267.97 31.1149 0)
       (effects (font (size 1.27 1.27)) (justify left))
     )
@@
   (symbol (lib_id "Device:C") (at 209.55 33.02 0) (unit 1)
     (in_bom yes) (on_board yes)
-    (property "Reference" "C33" (id 0) (at 210.82 31.1149 0)
+    (property "Reference" "C32" (id 0) (at 210.82 31.1149 0)
       (effects (font (size 1.27 1.27)) (justify left))
     )
@@
   (symbol (lib_id "Device:C") (at 132.08 26.67 0) (unit 1)
     (in_bom yes) (on_board yes)
-    (property "Reference" "C28" (id 0) (at 133.35 24.7649 0)
+    (property "Reference" "C27" (id 0) (at 133.35 24.7649 0)
       (effects (font (size 1.27 1.27)) (justify left))
     )
@@
   (symbol (lib_id "Device:C") (at 143.51 41.91 0) (unit 1)
     (in_bom yes) (on_board yes)
-    (property "Reference" "C30" (id 0) (at 137.541 39.4716 0)
+    (property "Reference" "C29" (id 0) (at 137.541 39.4716 0)
       (effects (font (size 1.27 1.27)) (justify left))
     )
@@
   (symbol (lib_id "Device:C") (at 33.02 125.73 270) (unit 1)
     (in_bom yes) (on_board yes)
-    (property "Reference" "C25" (id 0) (at 34.1884 119.761 0)
+    (property "Reference" "C24" (id 0) (at 34.1884 119.761 0)
       (effects (font (size 1.27 1.27)) (justify left))
     )
@@
   (symbol (lib_id "Device:C") (at 80.01 72.39 0) (unit 1)
     (in_bom yes) (on_board yes)
-    (property "Reference" "C27" (id 0) (at 81.28 70.4849 0)
+    (property "Reference" "C26" (id 0) (at 81.28 70.4849 0)
       (effects (font (size 1.27 1.27)) (justify left))
     )
@@
   (symbol (lib_id "Device:C") (at 243.84 33.02 0) (unit 1)
     (in_bom yes) (on_board yes)
-    (property "Reference" "C36" (id 0) (at 245.11 31.1149 0)
+    (property "Reference" "C35" (id 0) (at 245.11 31.1149 0)
       (effects (font (size 1.27 1.27)) (justify left))
     )
@@
   (symbol (lib_id "Device:C") (at 198.12 33.02 0) (unit 1)
     (in_bom yes) (on_board yes)
-    (property "Reference" "C31" (id 0) (at 199.39 31.1149 0)
+    (property "Reference" "C30" (id 0) (at 199.39 31.1149 0)
       (effects (font (size 1.27 1.27)) (justify left))
     )
@@
   (symbol (lib_id "Device:C") (at 143.51 26.67 0) (unit 1)
     (in_bom yes) (on_board yes)
-    (property "Reference" "C29" (id 0) (at 144.78 24.7649 0)
+    (property "Reference" "C28" (id 0) (at 144.78 24.7649 0)
       (effects (font (size 1.27 1.27)) (justify left))
     )
@@
   (symbol (lib_id "Device:R") (at 43.18 91.44 270) (unit 1)
     (in_bom yes) (on_board yes)
-    (property "Reference" "R38" (id 0) (at 43.18 86.1822 90))
+    (property "Reference" "R26" (id 0) (at 43.18 86.1822 90))
     (property "Value" "1k" (id 1) (at 43.18 88.4936 90))
     (property "Footprint" "Resistor_SMD:R_1206_3216Metric" (id 2) (at 43.18 89.662 90)
@@
   (symbol (lib_id "Device:R") (at 219.71 54.61 270) (unit 1)
     (in_bom yes) (on_board yes)
-    (property "Reference" "R41" (id 0) (at 219.71 56.9722 90))
+    (property "Reference" "R29" (id 0) (at 219.71 56.9722 90))
     (property "Value" "27" (id 1) (at 219.71 51.6636 90))
     (property "Footprint" "Resistor_SMD:R_0603_1608Metric" (id 2) (at 219.71 52.832 90)
@@
   (symbol (lib_id "Device:C") (at 220.98 33.02 0) (unit 1)
     (in_bom yes) (on_board yes)
-    (property "Reference" "C34" (id 0) (at 222.25 31.1149 0)
+    (property "Reference" "C33" (id 0) (at 222.25 31.1149 0)
       (effects (font (size 1.27 1.27)) (justify left))
     )
@@
   (symbol (lib_id "Device:R") (at 66.04 135.89 270) (unit 1)
     (in_bom yes) (on_board yes)
-    (property "Reference" "R40" (id 0) (at 66.04 130.6322 90))
+    (property "Reference" "R28" (id 0) (at 66.04 130.6322 90))
     (property "Value" "1k" (id 1) (at 66.04 132.9436 90))
     (property "Footprint" "Resistor_SMD:R_1206_3216Metric" (id 2) (at 66.04 134.112 90)
@@
   (symbol (lib_id "Memory_Flash:W25Q128JVS") (at 73.66 93.98 0) (unit 1)
     (in_bom yes) (on_board yes)
-    (property "Reference" "U20" (id 0) (at 64.77 83.82 0))
+    (property "Reference" "U19" (id 0) (at 64.77 83.82 0))
     (property "Value" "W25Q128JVS" (id 1) (at 81.28 104.14 0))
     (property "Footprint" "Package_SO:SOIC-8_5.23x5.23mm_P1.27mm" (id 2) (at 73.66 93.98 0)
@@
   (symbol (lib_id "Device:C") (at 232.41 33.02 0) (unit 1)
     (in_bom yes) (on_board yes)
-    (property "Reference" "C35" (id 0) (at 233.68 31.1149 0)
+    (property "Reference" "C34" (id 0) (at 233.68 31.1149 0)
       (effects (font (size 1.27 1.27)) (justify left))
     )
@@
   (symbol (lib_id "Device:C") (at 33.02 135.89 270) (unit 1)
     (in_bom yes) (on_board yes)
-    (property "Reference" "C26" (id 0) (at 34.1884 138.811 0)
+    (property "Reference" "C25" (id 0) (at 34.1884 138.811 0)
       (effects (font (size 1.27 1.27)) (justify left))
     )
@@
   (symbol (lib_id "Device:R") (at 58.42 76.2 0) (unit 1)
     (in_bom yes) (on_board yes)
-    (property "Reference" "R39" (id 0) (at 60.198 75.0316 0)
+    (property "Reference" "R27" (id 0) (at 60.198 75.0316 0)
       (effects (font (size 1.27 1.27)) (justify left))
     )
@@
   (symbol (lib_id "Device:R") (at 219.71 64.77 270) (unit 1)
     (in_bom yes) (on_board yes)
-    (property "Reference" "R42" (id 0) (at 219.71 67.1322 90))
+    (property "Reference" "R30" (id 0) (at 219.71 67.1322 90))
     (property "Value" "27" (id 1) (at 219.71 61.8236 90))
     (property "Footprint" "Resistor_SMD:R_0603_1608Metric" (id 2) (at 219.71 62.992 90)
@@
   (symbol (lib_id "Device:C") (at 255.27 33.02 0) (unit 1)
     (in_bom yes) (on_board yes)
-    (property "Reference" "C37" (id 0) (at 256.54 31.1149 0)
-      (effects (font (size 1.27 1.27)) (justify left))
-    )
+    (property "Reference" "C36" (id 0) (at 256.54 31.1149 0)
+      (effects (font (size 1.27 1.27)) (justify left))
+    )
