File: processors_all.kicad_sch (KiCad schematic)
At the start: 15 parts, among them SW1 TS-1187A-B-A-B, U17 74HC00, U18 74HCT595, U19 74HCT595

Commit message: Refactored top sheet
Parts:
- removed C22: 100n 50V, Capacitor_SMD:C_0402_1005Metric, symbol Device:C
- removed U17: 74HC00, symbol 74xx:74HC00
- renumbered C23 to C22, C24 to C23, R30 to R18, R31 to R19, R32 to R20, R33 to R21, R34 to R22, R35 to R23, R36 to R24, R37 to R25, U18 to U17, U19 to U18
Connections:
- no-connect marks 7 -> 1
Other:
- added sheet emergency_stop (emergency_stop.kicad_sch)
- note added: "To assert STEPPER_ENn, both the ESTOP from the button (hardware) and from the microcontroller (software) must be in the correct state"
